File: card.kicad_sch (KiCad schematic)
At the start: 13 parts, among them J3 Bus_Apple_II_Card_Side, U11 SN74LVC8T245, U12 SN74LVC8T245, U13 SN74LVC8T245, U14 SN74LVC8T245, U8 SN74LVC8T245, U9 SN74LVC8T245

Commit message: Moved routing to right side of FPGA
Connections:
- net RDY_3V3: now also U9.17 (B5); no longer U9.19 (B3)
- net RDY_5V: now also U9.7 (A5); no longer U9.5 (A3)
- net ~{I/O_STROBE}_3V3: now also U9.18 (B4); no longer U9.20 (B2)
- net ~{I/O_STROBE}_5V: now also U9.6 (A4); no longer U9.4 (A2)
- net ~{RES}_3V3: now also U9.19 (B3); no longer U9.21 (B1)
- net ~{RES}_5V: now also U9.5 (A3); no longer U9.3 (A1)
- no-connect marks 17 -> 16
Changed lines of the file:
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@@
 	)
 	(no_connect
-		(at 184.15 50.8)
-	)
-	(no_connect
-		(at 163.83 55.88)
-	)
-	(no_connect
-		(at 167.64 54.61)
+		(at 184.15 40.64)
 	)
 	(no_connect
@@
 	)
 	(no_connect
-		(at 184.15 55.88)
+		(at 163.83 40.64)
 	)
 	(no_connect
@@
 	)
 	(no_connect
-		(at 163.83 50.8)
-	)
-	(no_connect
 		(at 247.65 144.78)
 	)
@@
 	)
 	(no_connect
+		(at 184.15 35.56)
+	)
+	(no_connect
 		(at 55.88 73.66)
+	)
+	(no_connect
+		(at 163.83 35.56)
 	)
 	(no_connect
@@
 	(global_label "~{RES}_3V3"
 		(shape input)
-		(at 184.15 35.56 0)
-		(effects
-			(font
-				(size 1.27 1.27)
-			)
-			(justify left)
-		)
-		(property "Intersheetrefs" "${INTERSHEET_REFS}"
-			(at 184.15 35.56 90)
+		(at 184.15 45.72 0)
+		(effects
+			(font
+				(size 1.27 1.27)
+			)
+			(justify left)
+		)
+		(property "Intersheetrefs" "${INTERSHEET_REFS}"
+			(at 184.15 45.72 90)
 			(effects
 				(font
@@
 	(global_label "~{RES}_5V"
 		(shape input)
-		(at 163.83 35.56 180)
-		(effects
-			(font
-				(size 1.27 1.27)
-			)
-			(justify right)
-		)
-		(property "Intersheetrefs" "${INTERSHEET_REFS}"
-			(at 163.83 35.56 90)
+		(at 163.83 45.72 180)
+		(effects
+			(font
+				(size 1.27 1.27)
+			)
+			(justify right)
+		)
+		(property "Intersheetrefs" "${INTERSHEET_REFS}"
+			(at 163.83 45.72 90)
 			(effects
 				(font
@@
 	(global_label "RDY_5V"
 		(shape input)
-		(at 163.83 45.72 180)
-		(effects
-			(font
-				(size 1.27 1.27)
-			)
-			(justify right)
-		)
-		(property "Intersheetrefs" "${INTERSHEET_REFS}"
-			(at 163.83 45.72 90)
+		(at 163.83 55.88 180)
+		(effects
+			(font
+				(size 1.27 1.27)
+			)
+			(justify right)
+		)
+		(property "Intersheetrefs" "${INTERSHEET_REFS}"
+			(at 163.83 55.88 90)
 			(effects
 				(font
@@
 	(global_label "RDY_3V3"
 		(shape input)
-		(at 184.15 45.72 0)
-		(effects
-			(font
-				(size 1.27 1.27)
-			)
-			(justify left)
-		)
-		(property "Intersheetrefs" "${INTERSHEET_REFS}"
-			(at 184.15 45.72 90)
+		(at 184.15 55.88 0)
+		(effects
+			(font
+				(size 1.27 1.27)
+			)
+			(justify left)
+		)
+		(property "Intersheetrefs" "${INTERSHEET_REFS}"
+			(at 184.15 55.88 90)
 			(effects
 				(font
@@
 	(global_label "~{I{slash}O_STROBE}_3V3"
 		(shape input)
-		(at 184.15 40.64 0)
-		(effects
-			(font
-				(size 1.27 1.27)
-			)
-			(justify left)
-		)
-		(property "Intersheetrefs" "${INTERSHEET_REFS}"
-			(at 184.15 40.64 90)
+		(at 184.15 50.8 0)
+		(effects
+			(font
+				(size 1.27 1.27)
+			)
+			(justify left)
+		)
+		(property "Intersheetrefs" "${INTERSHEET_REFS}"
+			(at 184.15 50.8 90)
 			(effects
 				(font
@@
 	(global_label "~{I{slash}O_STROBE}_5V"
 		(shape input)
-		(at 163.83 40.64 180)
-		(effects
-			(font
-				(size 1.27 1.27)
-			)
-			(justify right)
-		)
-		(property "Intersheetrefs" "${INTERSHEET_REFS}"
-			(at 163.83 40.64 90)
-			(effects
-				(font
+		(at 163.83 50.8 180)
+		(effects
+			(font
+				(size 1.27 1.27)
+			)
+			(justify right)
+		)
+		(property "Intersheetrefs" "${INTERSHEET_REFS}"
+			(at 163.83 50.8 90)
+			(effects
+				(font

Commit message: Constraint Fixes
Connections:
- net ~{I/O_STROBE}_3V3: now also U9.20 (B2); no longer U9.18 (B4)
- net ~{I/O_STROBE}_5V: now also U9.4 (A2); no longer U9.6 (A4)
Changed lines of the file:
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@@
-	)
-	(no_connect
-		(at 184.15 40.64)
 	)
 	(no_connect
@@
 	)
 	(no_connect
-		(at 163.83 40.64)
-	)
-	(no_connect
 		(at 227.33 144.78)
 	)
@@
 	)
 	(no_connect
+		(at 184.15 50.8)
+	)
+	(no_connect
 		(at 247.65 129.54)
 	)
@@
 	(no_connect
 		(at 55.88 73.66)
+	)
+	(no_connect
+		(at 163.83 50.8)
 	)
 	(no_connect
@@
 	(global_label "~{I{slash}O_STROBE}_3V3"
 		(shape input)
-		(at 184.15 50.8 0)
-		(effects
-			(font
-				(size 1.27 1.27)
-			)
-			(justify left)
-		)
-		(property "Intersheetrefs" "${INTERSHEET_REFS}"
-			(at 184.15 50.8 90)
+		(at 184.15 40.64 0)
+		(effects
+			(font
+				(size 1.27 1.27)
+			)
+			(justify left)
+		)
+		(property "Intersheetrefs" "${INTERSHEET_REFS}"
+			(at 184.15 40.64 90)
 			(effects
 				(font
@@
 	(global_label "~{I{slash}O_STROBE}_5V"
 		(shape input)
-		(at 163.83 50.8 180)
-		(effects
-			(font
-				(size 1.27 1.27)
-			)
-			(justify right)
-		)
-		(property "Intersheetrefs" "${INTERSHEET_REFS}"
-			(at 163.83 50.8 90)
-			(effects
-				(font
+		(at 163.83 40.64 180)
+		(effects
+			(font
+				(size 1.27 1.27)
+			)
+			(justify right)
+		)
+		(property "Intersheetrefs" "${INTERSHEET_REFS}"
+			(at 163.83 40.64 90)
+			(effects
+				(font
