File: hardware/kicad/usb.kicad_sch (KiCad schematic)
At the start: 15 parts, among them J4 CONN_02X03, U1 LFE5U-25F-6BG381C, U6 FT231XQ

Commit message: Updates FPGA model in BOM and schematics
Replaces LFE5U-25F-6BG381C with LFE5U-85F-8BG381I in multiple files.
Ensures consistency across BOM, schematics, and PCB layouts for the updated FPGA model.
Adjusts related properties such as part number and connectivity attributes.

Addresses a hardware specification upgrade in branch 1.1.
Parts:
- U1: value LFE5U-25F-6BG381C -> LFE5U-85F-8BG381I; MPN LFE5U-85F-6BG381C -> LFE5U-85F-8BG381I
Changed lines of the file:
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@@
 			)
 		)
-		(property "Value" "LFE5U-25F-6BG381C"
+		(property "Value" "LFE5U-85F-8BG381I"
 			(at 113.03 50.8 0)
 			(effects
@@
 			)
 		)
-		(property "MPN" "LFE5U-85F-6BG381C"
+		(property "MPN" "LFE5U-85F-8BG381I"
 			(at 111.76 58.42 0)
 			(effects
