File: hardware/byte_ravn/kicad/byte_ravn.kicad_pcb (KiCad board)
At the start: 4 copper layers, 109.5 x 67.3 mm, 43 parts, among them J3 Bus_Apple_II_Card_Side, U11 SN74LVC8T245, U12 SN74LVC8T245, U13 SN74LVC8T245, U14 SN74LVC8T245, U5 TLV62569DBV, U8 SN74LVC8T245, U9 SN74LVC8T245

Commit message: Work in Progress - High Level Outline
Parts:
- added J1: Conn_01x16_Socket, Connector_PinHeader_2.54mm:PinHeader_1x16_P2.54mm_Horizontal, F.Cu at (187.5, 73.2)
- added J2: Conn_01x08_Socket, Connector_PinHeader_2.54mm:PinHeader_1x08_P2.54mm_Horizontal, F.Cu at (239.9, 67.8)
- added J4: Conn_01x05_Socket, Connector_PinHeader_2.54mm:PinHeader_1x05_P2.54mm_Horizontal, F.Cu at (213.6, 88.2)
- added J5: Conn_01x03_Socket, Connector_PinHeader_2.54mm:PinHeader_1x03_P2.54mm_Horizontal, F.Cu at (196.9, 87.8)
- added J6: Conn_01x03_Socket, Connector_PinHeader_2.54mm:PinHeader_1x03_P2.54mm_Horizontal, F.Cu at (185.3, 87.7)
- added J7: Conn_01x04_Socket, Connector_PinHeader_2.54mm:PinHeader_1x04_P2.54mm_Horizontal, F.Cu at (233.8, 83.6)
- added J8: Conn_01x04_Socket, Connector_PinHeader_2.54mm:PinHeader_1x04_P2.54mm_Horizontal, F.Cu at (258.4, 97.4)
- added J9: Conn_01x05_Socket, Connector_PinHeader_2.54mm:PinHeader_1x05_P2.54mm_Horizontal, F.Cu at (253.8, 86.5)
- moved C49 81.9 mm to (173.0, 84.4)
- moved C25 81.9 mm to (169.0, 74.4)
- moved C26 81.9 mm to (169.0, 76.9)
- moved C27 81.9 mm to (169.0, 79.4)
- moved C28 81.9 mm to (169.0, 81.9)
- moved C29 81.9 mm to (169.0, 84.4)
- moved C30 81.9 mm to (173.0, 74.4)
- moved C31 81.9 mm to (173.0, 76.9)
- moved C32 81.9 mm to (173.0, 79.4)
- moved C48 81.9 mm to (173.0, 81.9)
- moved C50 81.9 mm to (177.0, 74.4)
- moved C51 81.9 mm to (177.0, 76.9)
- moved C53 81.9 mm to (177.0, 79.4)
Other:
- board text added: "BR-1 5025 Robert Rico"
- board text removed: "BH-1-1 5025 Robert Rico"

Commit message: Updates to Ravn
Parts:
- removed C25, C26, C27, C28, C29, C30, C31, C32, C48, C49, C50, C51, C53: 22nF, Capacitor_SMD:C_0603_1608Metric
- removed J8: Conn_01x04_Socket, Connector_PinHeader_2.54mm:PinHeader_1x04_P2.54mm_Horizontal
- removed J9: Conn_01x05_Socket, Connector_PinHeader_2.54mm:PinHeader_1x05_P2.54mm_Horizontal
- J2: value Conn_01x08_Socket -> Conn_01x09_Socket; footprint Connector_PinHeader_2.54mm:PinHeader_1x08_P2.54mm_Horizontal -> Connector_PinHeader_2.54mm:PinHeader_1x09_P2.54mm_Horizontal
- J4: value Conn_01x05_Socket -> Conn_01x08_Socket; footprint Connector_PinHeader_2.54mm:PinHeader_1x05_P2.54mm_Horizontal -> Connector_PinHeader_2.54mm:PinHeader_1x08_P2.54mm_Horizontal
- J5: value Conn_01x03_Socket -> Conn_01x04_Socket; footprint Connector_PinHeader_2.54mm:PinHeader_1x03_P2.54mm_Horizontal -> Connector_PinHeader_2.54mm:PinHeader_1x04_P2.54mm_Horizontal
- J6: value Conn_01x03_Socket -> Conn_01x05_Socket; footprint Connector_PinHeader_2.54mm:PinHeader_1x03_P2.54mm_Horizontal -> Connector_PinHeader_2.54mm:PinHeader_1x05_P2.54mm_Horizontal
- J7: value Conn_01x04_Socket -> Conn_01x07_Socket; footprint Connector_PinHeader_2.54mm:PinHeader_1x04_P2.54mm_Horizontal -> Connector_PinHeader_2.54mm:PinHeader_1x07_P2.54mm_Horizontal
- moved J5 47.6 mm to (244.6, 88.3)
- moved J7 26.5 mm to (259.2, 91.1), turned to 0 degrees
- moved J6 13.4 mm to (174.9, 96.1)
- moved J1 5.75 mm to (193.0, 71.5)
- moved J2 3.38 mm to (240.3, 71.1)
- moved J4 0.52 mm to (213.2, 87.9)
Connections:
- J1 pad 1: unconnected-(J1-Pin_1-Pad1) -> A0_3V3
- J1 pad 10: unconnected-(J1-Pin_10-Pad10) -> A9_3V3
- J1 pad 11: unconnected-(J1-Pin_11-Pad11) -> A10_3V3
- J1 pad 12: unconnected-(J1-Pin_12-Pad12) -> A11_3V3
- J1 pad 13: unconnected-(J1-Pin_13-Pad13) -> A12_3V3
- J1 pad 14: unconnected-(J1-Pin_14-Pad14) -> A13_3V3
- J1 pad 15: unconnected-(J1-Pin_15-Pad15) -> A14_3V3
- J1 pad 16: unconnected-(J1-Pin_16-Pad16) -> A15_3V3
- J1 pad 2: unconnected-(J1-Pin_2-Pad2) -> A1_3V3
- J1 pad 3: unconnected-(J1-Pin_3-Pad3) -> A2_3V3
- J1 pad 4: unconnected-(J1-Pin_4-Pad4) -> A3_3V3
- J1 pad 5: unconnected-(J1-Pin_5-Pad5) -> A4_3V3
- J1 pad 6: unconnected-(J1-Pin_6-Pad6) -> A5_3V3
- J1 pad 7: unconnected-(J1-Pin_7-Pad7) -> A6_3V3
- J1 pad 8: unconnected-(J1-Pin_8-Pad8) -> A7_3V3
- J1 pad 9: unconnected-(J1-Pin_9-Pad9) -> A8_3V3
- J2 pad 1: unconnected-(J2-Pin_1-Pad1) -> R/~{W}_3V3
- J2 pad 2: unconnected-(J2-Pin_2-Pad2) -> D0_3V3
- J2 pad 3: unconnected-(J2-Pin_3-Pad3) -> D1_3V3
- J2 pad 4: unconnected-(J2-Pin_4-Pad4) -> D2_3V3
- J2 pad 5: unconnected-(J2-Pin_5-Pad5) -> D3_3V3
- J2 pad 6: unconnected-(J2-Pin_6-Pad6) -> D4_3V3
- J2 pad 7: unconnected-(J2-Pin_7-Pad7) -> D5_3V3
- J2 pad 8: unconnected-(J2-Pin_8-Pad8) -> D6_3V3
- J4 pad 1: unconnected-(J4-Pin_1-Pad1) -> ~{I/O_SELECT}_3V3
- J4 pad 2: unconnected-(J4-Pin_2-Pad2) -> PHI0_3V3
- J4 pad 3: unconnected-(J4-Pin_3-Pad3) -> µSync_3V3
- J4 pad 4: unconnected-(J4-Pin_4-Pad4) -> PHI1_3V3
- J4 pad 5: unconnected-(J4-Pin_5-Pad5) -> Q3_3V3
- J5 pad 1: unconnected-(J5-Pin_1-Pad1) -> RDY_3V3
- J5 pad 2: unconnected-(J5-Pin_2-Pad2) -> DMA_OUT_3V3
- J5 pad 3: unconnected-(J5-Pin_3-Pad3) -> INT_OUT_3V3
- J6 pad 1: unconnected-(J6-Pin_1-Pad1) -> GND
- J6 pad 2: unconnected-(J6-Pin_2-Pad2) -> CARD5V
- J6 pad 3: unconnected-(J6-Pin_3-Pad3) -> CARD12V
- J7 pad 1: unconnected-(J7-Pin_1-Pad1) -> ~{INH}_3V3
- J7 pad 2: unconnected-(J7-Pin_2-Pad2) -> ~{RES}_3V3
- J7 pad 3: unconnected-(J7-Pin_3-Pad3) -> ~{IRQ}_3V3
- J7 pad 4: unconnected-(J7-Pin_4-Pad4) -> ~{NMI}_3V3
Routing:
- net CARD-5V: track 0.00 -> 90.1 mm, vias 0 -> 1
- net CARD-12V: track 0.00 -> 88.6 mm, vias 0 -> 1
- net CARD12V: track 0.00 -> 46.0 mm
- net CARD5V: track 43.2 -> 77.8 mm
- net ~{DEVICE_SELECT}_3V3: track 29.5 -> 6.75 mm
- net DMA_IN_3V3: track 19.4 -> 0.99 mm
- net INT_IN_3V3: track 19.0 -> 1.28 mm
- net ~{DMA}_3V3: track 18.5 -> 1.57 mm
- net ~{I/O_SELECT}_3V3: track 18.4 -> 1.72 mm
- net A0_3V3: track 18.3 -> 2.01 mm
- net ~{NMI}_3V3: track 18.0 -> 1.86 mm
- net A1_3V3: track 18.3 -> 2.30 mm
- net A2_3V3: track 18.2 -> 2.59 mm
- net A3_3V3: track 18.2 -> 2.88 mm
- net ~{IRQ}_3V3: track 17.5 -> 2.15 mm
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