File: hardware/byte_ravn/kicad/power.kicad_sch (KiCad schematic)
At the start: 29 parts, among them U5 TLV62569DBV

Commit message: Updates to Ravn
Parts:
- removed C25, C26, C27, C28, C29, C30, C31, C32, C48, C49, C50, C51, C53: 22nF, Capacitor_SMD:C_0603_1608Metric, symbol Device:C
Other:
- note removed: "Capacitors near J1,2 connector"
