File: hardware/byte_hamr/kicad/card.kicad_sch (KiCad schematic)
At the start: 13 parts, among them J3 Bus_Apple_II_Card_Side, U11 SN74LVC8T245, U12 SN74LVC8T245, U13 SN74LVC8T245, U14 SN74LVC8T245, U8 SN74LVC8T245, U9 SN74LVC8T245

Commit message: Rev. 2
Parts:
- added U7: 74AHC1G04, SN74LVC1G04DBVR:SOT95P280X145-5N, symbol 74xGxx:74AHC1G04
Connections:
- net CARD5V: no longer C13.1, C14.1, C15.1, C18.1, C21.1, C36.1, U11.1 (V_{CCA}), U11.2 (DIR), U12.1 (V_{CCA}), U13.1 (V_{CCA}), U13.2 (DIR), U14.1 (V_{CCA}), U8.1 (V_{CCA}), U8.2 (DIR), U9.1 (V_{CCA}), U9.2 (DIR)
- net GND: now also U7.3 (GND); no longer U12.22 (~{OE})
- net R/~{W}_5V: now also U7.2; no longer U12.2 (DIR)
- net ~{RES}_5V: now also U13.8 (A6)
- net ~{RES}__READ_3V3: now reaches U13.16 (B6)
- new net +5V: C13.1, C14.1, C15.1, C18.1, C21.1, C36.1, U11.1 (V_{CCA}), U11.2 (DIR), U12.1 (V_{CCA}), U13.1 (V_{CCA}), U13.2 (DIR), U14.1 (V_{CCA}), U7.5 (VCC), U8.1 (V_{CCA}), U8.2 (DIR), U9.1 (V_{CCA}), U9.2 (DIR)
- new net DATA_OE: U12.22 (~{OE})
- new net INV_R/~{W}_5V: U12.2 (DIR), U7.4
- no-connect marks 4 -> 10

Commit message: Fabrication Feedback
Parts:
- U11, U12, U13, U14, U8, U9: MPN (none) -> SN74LVC8T245DBQR
- U7: MPN (none) -> SN74LVC1G04DBVR
Changed lines of the file:
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@@
 			)
 		)
-		(property "Datasheet" "https://www.ti.com/lit/ds/symlink/sn74lvc8t245.pdf"
+		(property "Datasheet" "https://www.ti.com/lit/ds/sces584c/sces584c.pdf?ts=1773424004893"
 			(at 173.99 88.9 0)
 			(effects
@@
 			)
 		)
-		(property "Description" "8-Bit Dual-Supply Bus Transceiver With Configurable Voltage Translation and 3-State Outputs"
+		(property "Description" "Translation Transceiver 1 Element 8 Bit per Element 3-State Output 24-SSOP"
+			(at 173.99 53.34 0)
+			(effects
+				(font
+					(size 1.27 1.27)
+				)
+				(hide yes)
+			)
+		)
+		(property "MPN" "SN74LVC8T245DBQR"
 			(at 173.99 53.34 0)
 			(effects
@@
 			)
 		)
-		(property "Datasheet" ""
+		(property "Datasheet" "https://yageogroup.com/content/datasheet/asset/file/DATASHEET_X2Y_SERIES_6-3V_TO_100V"
 			(at 21.59 186.69 0)
 			(effects
@@
 					(size 1.27 1.27)
 				)
+				(hide yes)
 			)
 		)
-		(property "Description" ""
+		(property "Description" "Surface-mount ceramicEMI filter capacitors"
 			(at 21.59 186.69 0)
 			(effects
@@
 					(size 1.27 1.27)
 				)
+				(hide yes)
 			)
 		)
@@
 			)
 		)
-		(property "Datasheet" ""
+		(property "Datasheet" "https://yageogroup.com/content/datasheet/asset/file/DATASHEET_X2Y_SERIES_6-3V_TO_100V"
 			(at 30.48 186.69 0)
 			(effects
@@
 					(size 1.27 1.27)
 				)
+				(hide yes)
 			)
 		)
-		(property "Description" ""
+		(property "Description" "Surface-mount ceramicEMI filter capacitors"
 			(at 30.48 186.69 0)
 			(effects
@@
 					(size 1.27 1.27)
 				)
+				(hide yes)
 			)
 		)
@@
 			)
 		)
-		(property "Datasheet" ""
+		(property "Datasheet" "https://yageogroup.com/content/datasheet/asset/file/DATASHEET_X2Y_SERIES_6-3V_TO_100V"
 			(at 66.04 186.69 0)
 			(effects
@@
 					(size 1.27 1.27)
 				)
+				(hide yes)
 			)
 		)
-		(property "Description" ""
+		(property "Description" "Surface-mount ceramicEMI filter capacitors"
 			(at 66.04 186.69 0)
 			(effects
@@
 					(size 1.27 1.27)
 				)
+				(hide yes)
 			)
 		)
@@
 			)
 		)
-		(property "Datasheet" "http://www.ti.com/lit/sg/scyt129e/scyt129e.pdf"
+		(property "Datasheet" "https://www.ti.com/lit/ds/symlink/sn74lvc1g04.pdf?ts=1753305682684&ref_url=https%253A%252F%252Fwww.ti.com%252Fproduct%252FSN74LVC1G04"
 			(at 46.99 148.59 0)
 			(effects
@@
 			)
 		)
-		(property "Description" "Single NOT Gate, Low-Voltage CMOS"
+		(property "Description" "Inverter IC 1 Channel SOT-23-5"
+			(at 46.99 148.59 0)
+			(effects
+				(font
+					(size 1.27 1.27)
+				)
+				(hide yes)
+			)
+		)
+		(property "MPN" "SN74LVC1G04DBVR"
 			(at 46.99 148.59 0)
 			(effects
@@
 			)
 		)
-		(property "Datasheet" "https://www.ti.com/lit/ds/symlink/sn74lvc8t245.pdf"
+		(property "Datasheet" "https://www.ti.com/lit/ds/sces584c/sces584c.pdf?ts=1773424004893"
 			(at 237.49 86.36 0)
 			(effects
@@
 			)
 		)
-		(property "Description" "8-Bit Dual-Supply Bus Transceiver With Configurable Voltage Translation and 3-State Outputs"
+		(property "Description" "Translation Transceiver 1 Element 8 Bit per Element 3-State Output 24-SSOP"
+			(at 237.49 50.8 0)
+			(effects
+				(font
+					(size 1.27 1.27)
+				)
+				(hide yes)
+			)
+		)
+		(property "MPN" "SN74LVC8T245DBQR"
 			(at 237.49 50.8 0)
 			(effects
@@
 			)
 		)
-		(property "Datasheet" "https://www.ti.com/lit/ds/symlink/sn74lvc8t245.pdf"
+		(property "Datasheet" "https://www.ti.com/lit/ds/sces584c/sces584c.pdf?ts=1773424004893"
 			(at 237.49 162.56 0)
 			(effects
@@
 			)
 		)
-		(property "Description" "8-Bit Dual-Supply Bus Transceiver With Configurable Voltage Translation and 3-State Outputs"
+		(property "Description" "Translation Transceiver 1 Element 8 Bit per Element 3-State Output 24-SSOP"
+			(at 237.49 127 0)
+			(effects
+				(font
+					(size 1.27 1.27)
+				)
+				(hide yes)
+			)
+		)
+		(property "MPN" "SN74LVC8T245DBQR"
 			(at 237.49 127 0)
 			(effects
@@
 			)
 		)
-		(property "Datasheet" "https://www.ti.com/lit/ds/symlink/sn74lvc8t245.pdf"
+		(property "Datasheet" "https://www.ti.com/lit/ds/sces584c/sces584c.pdf?ts=1773424004893"
 			(at 102.87 167.64 0)
 			(effects
@@
 			)
 		)
-		(property "Description" "8-Bit Dual-Supply Bus Transceiver With Configurable Voltage Translation and 3-State Outputs"
+		(property "Description" "Translation Transceiver 1 Element 8 Bit per Element 3-State Output 24-SSOP"
+			(at 102.87 132.08 0)
+			(effects
+				(font
+					(size 1.27 1.27)
+				)
+				(hide yes)
+			)
+		)
+		(property "MPN" "SN74LVC8T245DBQR"
 			(at 102.87 132.08 0)
 			(effects
@@
 			)
 		)
-		(property "Datasheet" ""
+		(property "Datasheet" "https://yageogroup.com/content/datasheet/asset/file/DATASHEET_X2Y_SERIES_6-3V_TO_100V"
 			(at 57.15 186.69 0)
 			(effects
@@
 					(size 1.27 1.27)
 				)
+				(hide yes)
 			)
 		)
-		(property "Description" ""
+		(property "Description" "Surface-mount ceramicEMI filter capacitors"
 			(at 57.15 186.69 0)
 			(effects
@@
 					(size 1.27 1.27)
 				)
+				(hide yes)
 			)
 		)
@@
 			)
 		)
-		(property "Datasheet" "https://www.ti.com/lit/ds/symlink/sn74lvc8t245.pdf"
+		(property "Datasheet" "https://www.ti.com/lit/ds/sces584c/sces584c.pdf?ts=1773424004893"
 			(at 172.72 165.1 0)
 			(effects
@@
 			)
 		)
-		(property "Description" "8-Bit Dual-Supply Bus Transceiver With Configurable Voltage Translation and 3-State Outputs"
+		(property "Description" "Translation Transceiver 1 Element 8 Bit per Element 3-State Output 24-SSOP"
+			(at 172.72 129.54 0)
+			(effects
+				(font
+					(size 1.27 1.27)
+				)
+				(hide yes)
+			)
+		)
+		(property "MPN" "SN74LVC8T245DBQR"
 			(at 172.72 129.54 0)
 			(effects
@@
 			)
 		)
-		(property "Datasheet" "https://www.ti.com/lit/ds/symlink/sn74lvc8t245.pdf"
+		(property "Datasheet" "https://www.ti.com/lit/ds/sces584c/sces584c.pdf?ts=1773424004893"
 			(at 101.6 88.9 0)
 			(effects
@@
 			)
 		)
-		(property "Description" "8-Bit Dual-Supply Bus Transceiver With Configurable Voltage Translation and 3-State Outputs"
+		(property "Description" "Translation Transceiver 1 Element 8 Bit per Element 3-State Output 24-SSOP"
+			(at 101.6 53.34 0)
+			(effects
+				(font
+					(size 1.27 1.27)
+				)
+				(hide yes)
+			)
+		)
+		(property "MPN" "SN74LVC8T245DBQR"
 			(at 101.6 53.34 0)
 			(effects
@@
 			)
 		)
-		(property "Datasheet" ""
+		(property "Datasheet" "https://yageogroup.com/content/datasheet/asset/file/DATASHEET_X2Y_SERIES_6-3V_TO_100V"
 			(at 39.37 186.69 0)
 			(effects
@@
 					(size 1.27 1.27)
 				)
+				(hide yes)
 			)
 		)
-		(property "Description" ""
+		(property "Description" "Surface-mount ceramicEMI filter capacitors"
 			(at 39.37 186.69 0)
 			(effects
@@
 					(size 1.27 1.27)
 				)
+				(hide yes)
 			)
 		)
@@
 			)
 		)
-		(property "Datasheet" ""
+		(property "Datasheet" "https://yageogroup.com/content/datasheet/asset/file/DATASHEET_X2Y_SERIES_6-3V_TO_100V"
 			(at 48.26 186.69 0)
 			(effects
@@
 					(size 1.27 1.27)
 				)
+				(hide yes)
 			)
 		)
-		(property "Description" ""
+		(property "Description" "Surface-mount ceramicEMI filter capacitors"
 			(at 48.26 186.69 0)
 			(effects
@@
 					(size 1.27 1.27)
 				)
+				(hide yes)
 			)
 		)
