File: hardware/byte_hamr/kicad/card_fpga.kicad_sch (KiCad schematic)
At the start: 3 parts, among them J1 Conn_01x13_Socket, U1 LFE5U-85F-8BG381I, Y1 FNETHE025

Commit message: Rev. 2
Parts:
- removed J1: Conn_01x13_Socket, Connector_PinHeader_2.54mm:PinHeader_1x13_P2.54mm_Horizontal, symbol Connector:Conn_01x13_Socket
- added J1: Conn_02x20_Odd_Even, Connector_PinHeader_2.54mm:PinHeader_2x20_P2.54mm_Vertical, symbol Connector_Generic:Conn_02x20_Odd_Even
- added J6: Conn_02x03_Odd_Even, Connector_PinHeader_2.54mm:PinHeader_2x03_P2.54mm_Vertical, symbol Connector_Generic:Conn_02x03_Odd_Even
- added R1, R2, R5, R6: 33Ω, Resistor_SMD:R_0603_1608Metric, symbol Device:R_Small
- Y1: value FNETHE025 -> 100Mhz; Datasheet-100 (none) -> https://www.digikey.com/en/products/detail/connor-winfield/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; MPN-100 (none) -> CWX813-100.0M
Connections:
- net +3V3: now also J6.6 (Pin_6)
- net GND: now also J1.1 (Pin_1), J1.11 (Pin_11), J1.13 (Pin_13), J1.15 (Pin_15), J1.17 (Pin_17), J1.19 (Pin_19), J1.21 (Pin_21), J1.23 (Pin_23), J1.25 (Pin_25), J1.27 (Pin_27), J1.29 (Pin_29), J1.3 (Pin_3), J1.31 (Pin_31), J1.33 (Pin_33), J1.35 (Pin_35), J1.37 (Pin_37), J1.39 (Pin_39), J1.5 (Pin_5), J1.7 (Pin_7), J1.9 (Pin_9), J6.5 (Pin_5)
- net I/O_PIN_1: now also U1.P3 (GPLL0T_IN), R1.2; no longer U1.L1 (PL65C)
- net I/O_PIN_10: now also U1.K2 (PL53A), J1.20 (Pin_20); no longer U1.A4 (PL11A)
- net I/O_PIN_11: now also U1.J1 (PL53B), R5.2; no longer U1.B5 (PL11C)
- net I/O_PIN_12: now also U1.H2 (PCLKT6_0), J1.24 (Pin_24); no longer U1.A5 (PL11B)
- net I/O_PIN_2: now also U1.P1 (PL92A), J1.4 (Pin_4); no longer U1.K1 (PL53D)
- net I/O_PIN_3: now also U1.P2 (PL92B), J1.6 (Pin_6); no longer U1.J1 (PL53B)
- net I/O_PIN_4: now also U1.N1 (PL89D), J1.8 (Pin_8); no longer U1.H1 (PL53C)
- net I/O_PIN_5: now also U1.M1 (PL89B), J1.10 (Pin_10); no longer U1.F2 (PCLKT7_0)
- net I/O_PIN_6: now also U1.L2 (PL86D), R2.2; no longer U1.E2 (PCLKC7_0)
- net I/O_PIN_7: now also U1.L1 (PL65C), J1.14 (Pin_14); no longer U1.E1 (PL38D)
- net I/O_PIN_8: now also U1.K3 (PL50D), J1.16 (Pin_16); no longer U1.D1 (PL38B)
- net I/O_PIN_9: now also U1.K1 (PL53D), J1.18 (Pin_18); no longer U1.C1 (PL38A)
- net I/O_PIN_20: now reaches U1.D2 (PL38C)
- net I/O_PIN_20: now also J1.40 (Pin_40)
- net CLK_100MHz: now reaches U1.F3 (PCLKC7_1)
- net CLK_100MHz: now also Y1.3
- net DATA_OE: now reaches U1.B20 (PT121B)
- net I/O_PIN_17: now reaches U1.F1 (PCLKC6_1)
- net I/O_PIN_17: now also J1.34 (Pin_34)
- net I/O_PIN_15: now reaches U1.G1 (PCLKC6_0)
- net I/O_PIN_15: now also J1.30 (Pin_30)
- net I/O_PIN_14: now reaches U1.G2 (PCLKT6_1)
- net I/O_PIN_14: now also J1.28 (Pin_28)
- net CLK_25MHz: no longer names the net of U1.G3 (PCLKT7_1)
- net CLK_25MHz: no longer Y1.3
- new net: J1.2 (Pin_2), R1.1
- new net: J1.12 (Pin_12), R2.1
- new net: J1.22 (Pin_22), R5.1
- new net: J1.32 (Pin_32), R6.1
- new net CARD-12V: J6.1 (Pin_1)
- new net CARD-5V: J6.4 (Pin_4)
- new net CARD12V: J6.2 (Pin_2)
- new net CARD5V: J6.3 (Pin_3)
- new net I/O_PIN_13: J1.26 (Pin_26), U1.H1 (PL53C)
- new net I/O_PIN_16: R6.2, U1.F2 (PCLKT7_0)
- new net I/O_PIN_18: J1.36 (Pin_36), U1.E2 (PCLKC7_0)
- new net I/O_PIN_19: J1.38 (Pin_38), U1.E1 (PL38D)
- new net ~{RES}__READ_3V3: U1.A5 (PL11B)
- no-connect marks 100 -> 91
Other:
- moved on the sheet: U1E

Commit message: Fabrication Feedback
Parts:
- R1, R2, R5, R6: MPN (none) -> 0603WAF330JT5E
- Y1: Datasheet-100 https://www.digikey.com/en/products/detail/connor-winfield/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 -> (none); Digike_y1 FNETHE025CT-ND -> (none); Digikey 3305-7050XOM2500BMD13CCC-CT-ND -> (none); Koncar FQ001 -> (none); LCSC C390569 -> (none); MNF1_URL www.diodes.com -> (none); MNF3_URL https://datasheet.lcsc.com/szlcsc/1912111437_Shenzhen-SCTF-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 -> (none); MPN FNETHE025 -> CWX813-100.0M; MPN-100 CWX813-100.0M -> (none); MPN2 SiT8008BC-81-33E-25.000000X -> (none); MPN3 S7D25.000000D20F30T -> (none); Mouse_r2 788-8008BC8133E25X -> (none); Mouser 729-FNETHE025 -> (none); Newark 80AC8624 -> (none); Side T -> (none); price100_Digikey 0.7942$ -> (none)
Changed lines of the file:
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@@
 			)
 		)
-		(property "Datasheet" "https://www.diodes.com/assets/Datasheets/FNETHE025.pdf"
+		(property "Datasheet" "https://www.digikey.com/en/products/detail/connor-winfield/CWX813-100-0M/695541"
 			(at 22.86 143.51 0)
 			(effects
@@
 			)
 		)
-		(property "Description" ""
-			(at 22.86 143.51 0)
-			(effects
-				(font
-					(size 1.27 1.27)
-				)
-			)
-		)
-		(property "Datasheet-100" "https://www.digikey.com/en/products/detail/connor-winfield/CWX813-100-0M/695541"
-			(at 22.86 143.51 0)
-			(effects
-				(font
-					(size 1.27 1.27)
-				)
-				(hide yes)
-			)
-		)
-		(property "MPN-100" "CWX813-100.0M"
-			(at 22.86 143.51 0)
-			(effects
-				(font
-					(size 1.27 1.27)
-				)
-				(hide yes)
-			)
-		)
-		(property "MNF1_URL" "www.diodes.com"
-			(at 22.86 143.51 0)
-			(effects
-				(font
-					(size 1.524 1.524)
-				)
-				(hide yes)
-			)
-		)
-		(property "MPN" "FNETHE025"
-			(at 22.86 143.51 0)
-			(effects
-				(font
-					(size 1.524 1.524)
-				)
-				(hide yes)
-			)
-		)
-		(property "MPN2" "SiT8008BC-81-33E-25.000000X"
-			(at 22.86 143.51 0)
-			(effects
-				(font
-					(size 1.27 1.27)
-				)
-				(hide yes)
-			)
-		)
-		(property "MNF3_URL" "https://datasheet.lcsc.com/szlcsc/1912111437_Shenzhen-SCTF-Elec-S7D25-000000D20F30T_C387026.pdf"
-			(at 22.86 143.51 0)
-			(effects
-				(font
-					(size 1.27 1.27)
-				)
-				(hide yes)
-			)
-		)
-		(property "MPN3" "S7D25.000000D20F30T"
-			(at 22.86 143.51 0)
-			(effects
-				(font
-					(size 1.27 1.27)
-				)
-				(hide yes)
-			)
-		)
-		(property "Mouser" "729-FNETHE025"
-			(at 22.86 143.51 0)
-			(effects
-				(font
-					(size 1.524 1.524)
-				)
-				(hide yes)
-			)
-		)
-		(property "Mouse_r2" "788-8008BC8133E25X "
-			(at 22.86 143.51 0)
-			(effects
-				(font
-					(size 1.27 1.27)
-				)
-				(hide yes)
-			)
-		)
-		(property "Digikey" "3305-7050XOM2500BMD13CCC-CT-ND"
-			(at 22.86 143.51 0)
-			(effects
-				(font
-					(size 1.27 1.27)
-				)
-				(hide yes)
-			)
-		)
-		(property "Digike_y1" "FNETHE025CT-ND"
+		(property "Description" "100 MHz XO (Standard) LVCMOS Oscillator 3.3V Enable/Disable 4-SMD, No Lead"
 			(at 22.86 143.51 0)
 			(effects
@@
 			)
 		)
-		(property "Newark" "80AC8624"
-			(at 22.86 143.51 0)
-			(effects
-				(font
-					(size 1.27 1.27)
-				)
-				(hide yes)
-			)
-		)
-		(property "LCSC" "C390569"
-			(at 22.86 143.51 0)
-			(effects
-				(font
-					(size 1.27 1.27)
-				)
-				(hide yes)
-			)
-		)
-		(property "price100_Digikey" "0.7942$"
-			(at 22.86 143.51 0)
-			(effects
-				(font
-					(size 1.27 1.27)
-				)
-				(hide yes)
-			)
-		)
-		(property "Koncar" "FQ001"
-			(at 22.86 143.51 0)
-			(effects
-				(font
-					(size 1.27 1.27)
-				)
-				(hide yes)
-			)
-		)
-		(property "Side" "T"
+		(property "MPN" "CWX813-100.0M"
 			(at 22.86 143.51 0)
 			(effects
@@
 			)
 		)
-		(property "Datasheet" "~"
+		(property "Datasheet" "https://www.royalohm.com/assets/pdf/products/smd/1.pdf"
 			(at 238.76 39.37 0)
 			(effects
@@
 			)
 		)
-		(property "Description" "Resistor, small symbol"
+		(property "Description" "Thick Film Resistors - SMD RMC 0603 1/10W 1% T/R-5000"
 			(at 238.76 39.37 0)
 			(effects
@@
 			)
 		)
+		(property "MPN" "0603WAF330JT5E"
+			(at 238.76 39.37 90)
+			(effects
+				(font
+					(size 1.27 1.27)
+				)
+				(hide yes)
+			)
+		)
 		(pin "1"
 		)
@@
 			)
 		)
-		(property "Datasheet" "http://www.latticesemi.com/~/media/LatticeSemi/Documents/DataSheets/ECP5/FPGA-DS-02012.pdf"
+		(property "Datasheet" "https://www.latticesemi.com/-/media/LatticeSemi/Documents/DataSheets/ECP5/FPGA-DS-02012-2-2-ECP5-ECP5G-Family-Data-Sheet.ashx?document_id=50461"
 			(at 26.67 19.05 0)
 			(effects
@@
 			)
 		)
-		(property "Description" ""
+		(property "Description" "ECP5 Field Programmable Gate Array (FPGA) IC 205 3833856 84000 381-FBGA"
 			(at 53.34 43.18 0)
 			(effects
@@
 					(size 1.27 1.27)
 				)
+				(hide yes)
 			)
 		)
@@
 			)
 		)
-		(property "Datasheet" "http://www.latticesemi.com/~/media/LatticeSemi/Documents/DataSheets/ECP5/FPGA-DS-02012.pdf"
+		(property "Datasheet" "https://www.latticesemi.com/-/media/LatticeSemi/Documents/DataSheets/ECP5/FPGA-DS-02012-2-2-ECP5-ECP5G-Family-Data-Sheet.ashx?document_id=50461"
 			(at 26.67 78.74 0)
 			(effects
@@
 			)
 		)
-		(property "Description" ""
+		(property "Description" "ECP5 Field Programmable Gate Array (FPGA) IC 205 3833856 84000 381-FBGA"
 			(at 53.34 102.87 0)
 			(effects
@@
 					(size 1.27 1.27)
 				)
+				(hide yes)
 			)
 		)
@@
 			)
 		)
-		(property "Datasheet" "http://www.latticesemi.com/~/media/LatticeSemi/Documents/DataSheets/ECP5/FPGA-DS-02012.pdf"
+		(property "Datasheet" "https://www.latticesemi.com/-/media/LatticeSemi/Documents/DataSheets/ECP5/FPGA-DS-02012-2-2-ECP5-ECP5G-Family-Data-Sheet.ashx?document_id=50461"
 			(at 229.87 107.95 0)
 			(effects
@@
 			)
 		)
-		(property "Description" ""
+		(property "Description" "ECP5 Field Programmable Gate Array (FPGA) IC 205 3833856 84000 381-FBGA"
 			(at 256.54 132.08 0)
 			(effects
@@
 					(size 1.27 1.27)
 				)
+				(hide yes)
 			)
 		)
@@
 			)
 		)
-		(property "Datasheet" "~"
+		(property "Datasheet" "https://www.royalohm.com/assets/pdf/products/smd/1.pdf"
 			(at 238.76 64.77 0)
 			(effects
@@
 			)
 		)
-		(property "Description" "Resistor, small symbol"
+		(property "Description" "Thick Film Resistors - SMD RMC 0603 1/10W 1% T/R-5000"
 			(at 238.76 64.77 0)
 			(effects
@@
 			)
 		)
+		(property "MPN" "0603WAF330JT5E"
+			(at 238.76 64.77 90)
+			(effects
+				(font
+					(size 1.27 1.27)
+				)
+				(hide yes)
+			)
+		)
 		(pin "1"
 		)
@@
 			)
 		)
-		(property "Datasheet" "~"
+		(property "Datasheet" "https://www.royalohm.com/assets/pdf/products/smd/1.pdf"
 			(at 238.76 77.47 0)
 			(effects
@@
 			)
 		)
-		(property "Description" "Resistor, small symbol"
+		(property "Description" "Thick Film Resistors - SMD RMC 0603 1/10W 1% T/R-5000"
 			(at 238.76 77.47 0)
 			(effects
@@
 			)
 		)
+		(property "MPN" "0603WAF330JT5E"
+			(at 238.76 77.47 90)
+			(effects
+				(font
+					(size 1.27 1.27)
+				)
+				(hide yes)
+			)
+		)
 		(pin "1"
 		)
@@
 			)
 		)
-		(property "Datasheet" "http://www.latticesemi.com/~/media/LatticeSemi/Documents/DataSheets/ECP5/FPGA-DS-02012.pdf"
+		(property "Datasheet" "https://www.latticesemi.com/-/media/LatticeSemi/Documents/DataSheets/ECP5/FPGA-DS-02012-2-2-ECP5-ECP5G-Family-Data-Sheet.ashx?document_id=50461"
 			(at 105.41 19.05 0)
 			(effects
@@
 			)
 		)
-		(property "Description" ""
+		(property "Description" "ECP5 Field Programmable Gate Array (FPGA) IC 205 3833856 84000 381-FBGA"
 			(at 132.08 43.18 0)
 			(effects
@@
 					(size 1.27 1.27)
 				)
+				(hide yes)
 			)
 		)
@@
 			)
 		)
-		(property "Datasheet" "~"
+		(property "Datasheet" "https://www.royalohm.com/assets/pdf/products/smd/1.pdf"
 			(at 238.76 52.07 0)
 			(effects
@@
 			)
 		)
-		(property "Description" "Resistor, small symbol"
+		(property "Description" "Thick Film Resistors - SMD RMC 0603 1/10W 1% T/R-5000"
 			(at 238.76 52.07 0)
 			(effects
@@
 			)
 		)
+		(property "MPN" "0603WAF330JT5E"
+			(at 238.76 52.07 90)
+			(effects
+				(font
+					(size 1.27 1.27)
+				)
+				(hide yes)
+			)
+		)
 		(pin "1"
 		)
@@
 			)
 		)
-		(property "Datasheet" "http://www.latticesemi.com/~/media/LatticeSemi/Documents/DataSheets/ECP5/FPGA-DS-02012.pdf"
+		(property "Datasheet" "https://www.latticesemi.com/-/media/LatticeSemi/Documents/DataSheets/ECP5/FPGA-DS-02012-2-2-ECP5-ECP5G-Family-Data-Sheet.ashx?document_id=50461"
 			(at 106.68 80.01 0)
 			(effects
@@
 			)
 		)
-		(property "Description" ""
+		(property "Description" "ECP5 Field Programmable Gate Array (FPGA) IC 205 3833856 84000 381-FBGA"
 			(at 133.35 104.14 0)
 			(effects
@@
 					(size 1.27 1.27)
 				)
+				(hide yes)
 			)
 		)
