File: hardware/byte_hamr/kicad/flash.kicad_sch (KiCad schematic)
At the start: 11 parts, among them U1 LFE5U-85F-8BG381I, U10 IS25LP128F-JBLE

Commit message: Rev. 2
Connections:
- no-connect marks 1 -> 5
Changed lines of the file:
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@@
 		(at 220.98 107.95)
+	)
+	(no_connect
+		(at 182.88 95.25)
+	)
+	(no_connect
+		(at 182.88 97.79)
+	)
+	(no_connect
+		(at 220.98 95.25)
+	)
+	(no_connect
+		(at 220.98 97.79)
 	)
 	(wire

Commit message: Fabrication Feedback
Parts:
- R11: Digikey 311-10KLMCT-ND -> (none); Koncar FR013 -> (none); LCSC C15401 -> (none); MNF1_URL www.yageo.com -> (none); MPN RC0603FR-0710KL -> AF0603FR-0710KL; Mouser 603-RC0603FR-0710KL -> (none); Newark 94X1379 -> (none)
- R12, R27, R28: MPN (none) -> AF0603FR-0710KL
- R29: MPN (none) -> 0603WAF1101T5E
- R30: MNF1_URL www.yageo.com -> (none)
- R31, R32, R33: MPN (none) -> RC0603FR-0715KL
- U10: Datasheet2 http://www.issi.com/WW/pdf/25LP-WP032D.pdf -> (none); Digike_y2 IS25LP128F-JBLE-ND -> (none); Digike_y3 706-1607-1-ND -> (none); Digikey W25Q128JVSIQCT-ND -> (none); Dtasheet4 https://www.winbond.com/resource-files/w25q128jv%20spi%20re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 -> (none); Koncar FU003 -> (none); LCSC C113767 -> (none); LowCost 870-IS25LP032DJBLETR -> (none); MNF1_URL www.issi.com -> (none); MNF2_URL www.issi.com -> (none); MNF3_URL www.issi.com -> (none); MNF4_URL www.winbond.com -> (none); MPN2 IS25LP032D-JNLE-TR -> (none); MPN3 IS25LP032D-JNLA3 -> (none); MPN4 W25Q128JVSIM -> (none); Mouse_1r 727-S25FL128LAMFV013 -> (none); Mouse_r3 454-W25Q128JVSIQTR -> (none); Mouser 454-W25Q128JVSIMTR -> (none); Newark 38AC3510 -> (none); price100_LCSC 0.7796$ -> (none)
