File: hardware/byte_hamr/kicad/ram.kicad_sch (KiCad schematic)
At the start: 7 parts, among them U1 LFE5U-85F-8BG381I, U2 MT48LC16M16A2TG

Commit message: Fabrication Feedback
Parts:
- C16: MPN (none) -> CL21B225KOFNNNE
- U2: Datasheet4 https://www.alliancememory.com/wp-content/uploads/pdf/dram/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 -> (none); Digike_y2 1450-1352-1-ND -> (none); Digikey 1450-1385-1-ND -> (none); Koncar FU007 -> (none); LCSC C492195 -> (none); LCS_C1 C524867 -> (none); MFG1 Micron -> (none); MFG2 ISSI -> (none); MFG3 Winbond -> (none); MFG4 Alliance -> (none); MNF1_URL www.micron.com -> (none); MNF2_URL www.issi.com -> (none); MPN MT48LC16M16A2TG-6A -> AS4C32M16SB-7TCNTR; MPN2 IS42S16160G-7TL-TR -> (none); MPN4 AS4C32M16SB-7TCN -> (none); MPN5 M12L2561616A-6TG2T -> (none); MP_N3 W9812G6KH-6 -> (none); Mouse_r0 913-AS4C32M16SB-7TCN -> (none); Mouse_r1 913-4C16M16SA-6TCNTR -> (none); Mouse_r2 913-4816M16A2TG6AGTR -> (none); Mouse_r3 870-42S16320F7TL -> (none); Mouse_r4 454-W9825G6KH-5 -> (none); Mouse_r5 454-W9825G6KH-6 -> (none); Mouse_r6 340-128308-REEL -> (none); Mouse_r7 870-IS42S16160G7TLTR -> (none); Mouser 870-IS42S16160G7TLTR -> (none); Side T -> (none); price100_Mouse_r 2.3€ -> (none); price500_LCSC 0.9227$ -> (none)
