File: hardware/byte_hamr/kicad/project_byte_hamr.kicad_pcb (KiCad board)
At the start: 4 copper layers, 109.5 x 67.3 mm, 95 parts, among them J1 Conn_01x13_Socket, J3 Bus_Apple_II_Card_Side, J4 CONN_02X03, U1 LFE5U-85F-8BG381I, U10 IS25LP128F-JBLE, U11 SN74LVC8T245, U12 SN74LVC8T245, U13 SN74LVC8T245, U14 SN74LVC8T245, U2 MT48LC16M16A2TG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

Commit message: Improves signal check functionality and testability
Refactors the signal check gateware for enhanced functionality and testability.

This commit introduces a fake PHI0 generator, enabling standalone
testing of the GPIO3 activity indicator without requiring an
external Apple II connection. An external PHI0 detector
automatically switches to the fake clock when no external clock
source is present.

The heartbeat LED is changed to a 250kHz square wave for easier
oscilloscope testing.

Pull-up resistors are enabled on the Apple II I/O signals.

A diode rotation is corrected on the PCB.
Parts:
- turned D1 to 90 degrees
- turned D2 to -90 degrees
Connections:
- D1 pad 1: USB5V -> +5V
- D1 pad 2: +5V -> USB5V
- D2 pad 1: CARD5V -> +5V
- D2 pad 2: +5V -> CARD5V

Commit message: Rev. 2
Parts:
- removed D19: RED, LED_SMD:LED_0805_2012Metric
- removed D3: YELLOW, LED_SMD:LED_0805_2012Metric
- removed H1, H2, H3, H4: MountingHole_Pad, MountingHole:MountingHole_3mm_Pad
- removed R37: 549, Resistor_SMD:R_0603_1608Metric
- added J6: Conn_02x03_Odd_Even, Connector_PinHeader_2.54mm:PinHeader_2x03_P2.54mm_Vertical, F.Cu at (233.0, 115.2)
- added R2: 33Ω, Resistor_SMD:R_0603_1608Metric, F.Cu at (226.7, 71.0)
- added R5: 33Ω, Resistor_SMD:R_0603_1608Metric, F.Cu at (226.7, 83.9)
- added R6: 33Ω, Resistor_SMD:R_0603_1608Metric, F.Cu at (226.7, 96.5)
- added U7: 74AHC1G04, SN74LVC1G04DBVR:SOT95P280X145-5N, B.Cu at (195.7, 110.0)
- J1: value Conn_01x13_Socket -> Conn_02x20_Odd_Even; footprint Connector_PinHeader_2.54mm:PinHeader_1x13_P2.54mm_Horizontal -> Connector_PinHeader_2.54mm:PinHeader_2x20_P2.54mm_Vertical
- R1: value 549 -> 33Ω
- Y1: value FNETHE025 -> 100Mhz
- moved R9 49.8 mm to (193.2, 62.0), turned to 90 degrees
- moved C48 49.2 mm to (205.6, 61.2)
- moved U6 45.8 mm to (192.2, 66.4), turned to 90 degrees
- moved R49 45.4 mm to (196.9, 66.0), turned to 0 degrees
- moved C16 45.0 mm to (196.9, 67.8), turned to 180 degrees
- moved R11 44.7 mm to (208.2, 69.0)
- moved Y1 43.9 mm to (206.8, 94.1), turned to 0 degrees
- moved R27 43.8 mm to (207.5, 59.7)
- moved R50 42.6 mm to (196.9, 64.2), turned to 0 degrees
- moved C35 41.5 mm to (198.9, 95.2), turned to 0 degrees
- moved J1 39.7 mm to (220.7, 58.3)
- moved R28 39.3 mm to (211.2, 69.0)
- moved U10 38.3 mm to (210.8, 64.5), turned to 180 degrees
- moved D2 37.9 mm to (224.9, 114.2)
- moved R29 37.8 mm to (210.6, 59.7)
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Connections:
- C13 pad 1: CARD5V -> +5V
- C14 pad 1: CARD5V -> +5V
- C15 pad 1: CARD5V -> +5V
- C18 pad 1: CARD5V -> +5V
- C21 pad 1: CARD5V -> +5V
- C36 pad 1: CARD5V -> +5V
- J1 pad 1: I/O_PIN_1 -> GND
- J1 pad 10: I/O_PIN_10 -> I/O_PIN_5
- J1 pad 11: I/O_PIN_11 -> GND
- J1 pad 12: I/O_PIN_12 -> Net-(J1-Pin_12)
- J1 pad 2: I/O_PIN_2 -> Net-(J1-Pin_2)
- J1 pad 3: I/O_PIN_3 -> GND
- J1 pad 4: I/O_PIN_4 -> I/O_PIN_2
- J1 pad 5: I/O_PIN_5 -> GND
- J1 pad 6: I/O_PIN_6 -> I/O_PIN_3
- J1 pad 7: I/O_PIN_7 -> GND
- J1 pad 8: I/O_PIN_8 -> I/O_PIN_4
- J1 pad 9: I/O_PIN_9 -> GND
- R1 pad 1: FTDI_nRXLED -> Net-(J1-Pin_2)
- R1 pad 2: Net-(D3-K) -> I/O_PIN_1
- U1 pad A4: I/O_PIN_10 -> unconnected-(U1F-PL11A-PadA4)
- U1 pad A5: I/O_PIN_12 -> ~{RES}__READ_3V3
- U1 pad B20: unconnected-(U1B-PT121B-PadB20) -> DATA_OE
- U1 pad B5: I/O_PIN_11 -> unconnected-(U1F-PL11C-PadB5)
- U1 pad C1: I/O_PIN_9 -> unconnected-(U1F-PL38A-PadC1)
- U1 pad D1: I/O_PIN_8 -> unconnected-(U1F-PL38B-PadD1)
- U1 pad D2: unconnected-(U1F-PL38C-PadD2) -> I/O_PIN_20
- U1 pad E1: I/O_PIN_7 -> I/O_PIN_19
- U1 pad E2: I/O_PIN_6 -> I/O_PIN_18
- U1 pad F1: unconnected-(U1E-PCLKC6_1-PadF1) -> I/O_PIN_17
- U1 pad F2: I/O_PIN_5 -> I/O_PIN_16
- U1 pad F3: unconnected-(U1F-PCLKC7_1-PadF3) -> CLK_100MHz
- U1 pad G1: unconnected-(U1E-PCLKC6_0-PadG1) -> I/O_PIN_15
- U1 pad G2: unconnected-(U1E-PCLKT6_1-PadG2) -> I/O_PIN_14
- U1 pad G3: CLK_25MHz -> unconnected-(U1F-PCLKT7_1-PadG3)
- U1 pad H1: I/O_PIN_4 -> I/O_PIN_13
- U1 pad H2: unconnected-(U1E-PCLKT6_0-PadH2) -> I/O_PIN_12
- U1 pad J1: I/O_PIN_3 -> I/O_PIN_11
- U1 pad K1: I/O_PIN_2 -> I/O_PIN_9
- U1 pad K2: unconnected-(U1E-PL53A-PadK2) -> I/O_PIN_10
- U1 pad K3: unconnected-(U1E-PL50D-PadK3) -> I/O_PIN_8
- U1 pad L1: I/O_PIN_1 -> I/O_PIN_7
- U1 pad L2: unconnected-(U1E-PL86D-PadL2) -> I/O_PIN_6
- U1 pad M1: unconnected-(U1E-PL89B-PadM1) -> I/O_PIN_5
- U1 pad N1: unconnected-(U1E-PL89D-PadN1) -> I/O_PIN_4
- U1 pad P1: unconnected-(U1E-PL92A-PadP1) -> I/O_PIN_2
- U1 pad P2: unconnected-(U1E-PL92B-PadP2) -> I/O_PIN_3
- U1 pad P3: unconnected-(U1E-GPLL0T_IN-PadP3) -> I/O_PIN_1
- U11 pad 1: CARD5V -> +5V
- U11 pad 2: CARD5V -> +5V
- U12 pad 1: CARD5V -> +5V
- U12 pad 2: R/~{W}_5V -> INV_R/~{W}_5V
- U12 pad 22: GND -> DATA_OE
- U13 pad 1: CARD5V -> +5V
- U13 pad 16: unconnected-(U13-B6-Pad16) -> ~{RES}__READ_3V3
- U13 pad 2: CARD5V -> +5V
- U13 pad 8: unconnected-(U13-A6-Pad8) -> ~{RES}_5V
- U14 pad 1: CARD5V -> +5V
- U6 pad 10: FT3V3OUT -> unconnected-(U6-3V3OUT-Pad10)
- U6 pad 14: FTDI_nRXLED -> unconnected-(U6-CBUS1-Pad14)
- U6 pad 7: FTDI_nTXLED -> unconnected-(U6-CBUS2-Pad7)
- U8 pad 1: CARD5V -> +5V
- U8 pad 2: CARD5V -> +5V
- U9 pad 1: CARD5V -> +5V
- U9 pad 2: CARD5V -> +5V
- Y1 pad 3: CLK_25MHz -> CLK_100MHz
Routing:
- net CARD12V: track 0.00 -> 73.6 mm, vias 0 -> 1
- net I/O_PIN_20: track 0.00 -> 37.1 mm, vias 0 -> 1
- net I/O_PIN_19: track 0.00 -> 34.7 mm
- net I/O_PIN_16: track 0.00 -> 34.4 mm, vias 0 -> 2
- net I/O_PIN_18: track 0.00 -> 33.5 mm, vias 0 -> 1
- net CARD-5V: track 0.00 -> 32.2 mm
- net CARD-12V: track 0.00 -> 31.2 mm
- net I/O_PIN_17: track 0.00 -> 30.7 mm
- net /usb/FTD+: track 16.4 -> 45.2 mm
- net ~{RES}__READ_3V3: track 0.00 -> 28.6 mm, vias 0 -> 2
- net /usb/FTD-: track 18.4 -> 46.4 mm
- net I/O_PIN_15: track 0.00 -> 26.6 mm
- net +5V: track 52.4 -> 78.8 mm, vias 7 -> 12
- net I/O_PIN_14: track 0.00 -> 25.7 mm, vias 0 -> 1
- net CARD5V: track 43.2 -> 19.2 mm, vias 8 -> 0
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- removed copper zone on In2.Cu, net CARD5V
Other:
- board size 109.5 x 67.3 mm -> 103.8 x 67.3 mm
- board text added: "1"
- board text added: "20"
- board text added: "BH-2-0 1126 Robert Rico"
- board text added: "GND"
- board text added: "Rev. 2.0"
- board text removed: "BH-1-1 5025 Robert Rico"
- board text removed: "Rev. 1.1"

Commit message: Fabrication Feedback
Routing:
- net GND: track 342.3 -> 343.2 mm
